File: hardware/QuadPreRecorder.kicad_sch (KiCad schematic)
At the start: 180 parts, among them J1 9V DC IN, J2 AMBISONIC MIC RJ45, J3 MSP3520 TFT 3.5IN 14PIN HEADER, J4 1/4in BINAURAL LINE OUT, J5 1/8in BINAURAL HEADPHONE OUT, J6 ANALOG TEST HEADER 2x13, J7 DIGITAL TEST HEADER 2x13, SW1 PAD -10dB, SW2 RECORD START/STOP, SW3 MASTER GAIN, SW4 TFT MENU NAV, U1 TPS62160DGK, U10 TPA6132A2, U2 TPS7A2033PDBV, U3 TLE2426ID, U4 CD4053BPW, U5 CD4053BPW, U6 OPA1654, U7 PCM1864DBT, U8 Teensy 4.1, U9 PCM5102A

Commit message: Rev B through Rev C3: 1590XX enclosure, CAT6 mic input, mic-mode rebuild, fab package, 3D enclosure models
- Rev B 2-layer, then Rev C/C2/C3 on Hammond 1590XX: USB-C power/data, capacitive MSP3526, TPA6130A2 headphone amp, LiPo + BQ24074, SW4 5-way encoder
- Mic-mode rebuild: per-channel bias off/5V/9V, cold-leg grounding, balanced inputs, SPICE CMRR fixes
- Enclosure fit recheck applied (J4/J5/J9 moves, SW2 replacement, front-wall LEDs); ADC test points; ADP7142 LDO swap
- PCBWay Rev C3 handoff package with 4-layer gerbers, BOM/CPL, best-source pricing
- Interactive labeled 3D enclosure models (1590XX as-built with logo + 1590F concept), labeled-views PDF, blog embed notes

Co-Authored-By: Claude Fable 5 <noreply@anthropic.com>
Claude-Session: https://claude.ai/code/session_01CTGyPyq5ASmP2zYeDmwtXd
Parts:
- removed C19, C27: 4.7uF 16V, Capacitor_SMD:C_1206_3216Metric, symbol Device:C
- removed C23: 22pF C0G, Capacitor_SMD:C_0603_1608Metric, symbol Device:C
- removed R16: 1M, Resistor_SMD:R_0603_1608Metric, symbol Device:R
- removed R22: 68k 0.1%, Resistor_SMD:R_0603_1608Metric, symbol Device:R
- removed R23: 33k 0.1%, Resistor_SMD:R_0603_1608Metric, symbol Device:R
- removed R28: 10k 0.1%, Resistor_SMD:R_0603_1608Metric, symbol Device:R
- removed R32: 90.9k 0.1%, Resistor_SMD:R_0603_1608Metric, symbol Device:R
- removed R36: 100R, Resistor_SMD:R_0603_1608Metric, symbol Device:R
- added C100: 100pF C0G, Capacitor_SMD:C_0603_1608Metric, symbol Device:C
- added C104, C28: 4.7uF 35V FILM, Capacitor_SMD:C_1812_4532Metric, symbol Device:C
- added C108: 22pF C0G, Capacitor_SMD:C_0603_1608Metric, symbol Device:C
- added C109, C110, C33, C34, C35, C36, C40, C41, C43, C44, C47, C50, C54, C56, C64, C69, C70, C71, C72, C73: 100nF, Capacitor_SMD:C_0603_1608Metric, symbol Device:C
- added C32: 10nF C0G, Capacitor_SMD:C_0603_1608Metric, symbol Device:C
- added C37: 10uF 16V, Capacitor_SMD:C_1206_3216Metric, symbol Device:C
- added C39: 1uF, Capacitor_SMD:C_0805_2012Metric, symbol Device:C
- added C42, C45, C46, C55, C62: 10uF, Capacitor_SMD:C_1206_3216Metric, symbol Device:C
- added C48, C49, C93, C94: 10nF, Capacitor_SMD:C_0603_1608Metric, symbol Device:C
- added C51, C52: 2.2uF, Capacitor_SMD:C_0805_2012Metric, symbol Device:C
- added C53, C59, C60, C61, C65: 1uF, Capacitor_SMD:C_0603_1608Metric, symbol Device:C
- added C57, C58, C86, C87: 2.2uF 25V FILM, Capacitor_SMD:C_1210_3225Metric, symbol Device:C
- added C67, C68: 2.2nF C0G, Capacitor_SMD:C_0603_1608Metric, symbol Device:C
- added C79: 47nF, Capacitor_SMD:C_0603_1608Metric, symbol Device:C
- added C80: 4.7nF C0G, Capacitor_SMD:C_0603_1608Metric, symbol Device:C
- added C81: 47pF C0G, Capacitor_SMD:C_0603_1608Metric, symbol Device:C
- added D13: 1N4148W, Diode_SMD:D_SOD-123, symbol Device:D_Small
- added D3: SS14, Diode_SMD:D_SMA, symbol Device:D_Schottky
- added D4: POWER BLUE, LED_THT:LED_D3.0mm_Horizontal_O1.27mm_Z6.0mm, symbol Device:LED
- added D5: RECORD RED, LED_THT:LED_D3.0mm_Horizontal_O1.27mm_Z6.0mm, symbol Device:LED
- added J3: MSP3526 TFT 3.5IN 14PIN SOCKET, Connector_PinSocket_2.54mm:PinSocket_1x14_P2.54mm_Vertical, symbol Connector_Generic:Conn_01x14
- added J4: 1/4in BINAURAL LINE OUT, Connector_Audio:Jack_6.35mm_Neutrik_NRJ6HF_Horizontal, symbol Connector_Audio:AudioJack3
- added J5: 1/8in BINAURAL HEADPHONE OUT, Connector_Audio:Jack_3.5mm_CUI_SJ1-3533NG_Horizontal, symbol Connector_Audio:AudioJack3
- added K1: G6K-2F-Y 5VDC, Relay_SMD:Relay_DPDT_Omron_G6K-2F-Y, symbol Relay:G6K-2
- added Q1, Q2, Q5: 2N7002, Package_TO_SOT_SMD:SOT-23, symbol Transistor_FET:Q_NMOS_GSD
- added R106, R50, R51, R52, R53, R60, R70, R71, R72, R73, R74, R79, R83, R96, R97: 10k, Resistor_SMD:R_0603_1608Metric, symbol Device:R
- added R107, R37, R42, R61, R84: 100R, Resistor_SMD:R_0603_1608Metric, symbol Device:R
- added R108, R129, R41, R43, R64, R85: 100k, Resistor_SMD:R_0603_1608Metric, symbol Device:R
- added R113: 100R RF, Resistor_SMD:R_0603_1608Metric, symbol Device:R
- added R117: 1M, Resistor_SMD:R_0603_1608Metric, symbol Device:R
- added R121: 10k 0.1%, Resistor_SMD:R_0603_1608Metric, symbol Device:R
- added R125: 90.9k 0.1%, Resistor_SMD:R_0603_1608Metric, symbol Device:R
- added R130: 130k, Resistor_SMD:R_0603_1608Metric, symbol Device:R
- added R44, R45: 4.7k, Resistor_SMD:R_0603_1608Metric, symbol Device:R
- added R46, R47, R48, R49, R57, R58, R59, R69: 33R, Resistor_SMD:R_0603_1608Metric, symbol Device:R
- added R54: 2.2k, Resistor_SMD:R_0603_1608Metric, symbol Device:R
- added R55: 1k, Resistor_SMD:R_0603_1608Metric, symbol Device:R
- added R56: 100R TFT BACKLIGHT, Resistor_SMD:R_0805_2012Metric, symbol Device:R
- added R62, R63: 470R, Resistor_SMD:R_0603_1608Metric, symbol Device:R
- added R65, R66: 10R, Resistor_SMD:R_0603_1608Metric, symbol Device:R
- added R82: 80.6k, Resistor_SMD:R_0603_1608Metric, symbol Device:R
- added SW2: RECORD START/STOP, Button_Switch_THT:SW_PUSH_6mm, symbol Switch:SW_Push
- added SW3: MASTER GAIN, Rotary_Encoder:RotaryEncoder_Alps_EC11E-Switch_Vertical_H20mm, symbol Device:RotaryEncoder_Switch
- added SW4: TFT MENU NAV, QuadPreRecorder:SW_Nav5_ALPS_RKJXT1F42001, symbol QuadPreRecorder:SW_Nav5
- added TP10: DAC_LRCLK, TestPoint:TestPoint_Pad_1.5x1.5mm, symbol Connector:TestPoint
- added TP11: DAC_DIN, TestPoint:TestPoint_Pad_1.5x1.5mm, symbol Connector:TestPoint
- added TP12: +3V3_DC, TestPoint:TestPoint_Pad_1.5x1.5mm, symbol Connector:TestPoint
- added TP13, TP14, TP8: GND, TestPoint:TestPoint_Pad_1.5x1.5mm, symbol Connector:TestPoint
- added TP3: ADC_MCLK, TestPoint:TestPoint_Pad_1.5x1.5mm, symbol Connector:TestPoint
- added TP4: ADC_BCLK, TestPoint:TestPoint_Pad_1.5x1.5mm, symbol Connector:TestPoint
- added TP5: ADC_LRCLK, TestPoint:TestPoint_Pad_1.5x1.5mm, symbol Connector:TestPoint
- added TP6: ADC_TDM, TestPoint:TestPoint_Pad_1.5x1.5mm, symbol Connector:TestPoint
- added TP7: ADC_DOUT2, TestPoint:TestPoint_Pad_1.5x1.5mm, symbol Connector:TestPoint
- added TP9: DAC_BCLK, TestPoint:TestPoint_Pad_1.5x1.5mm, symbol Connector:TestPoint
- added U10: TPA6130A2RTJ, Package_DFN_QFN:WQFN-20-1EP_4x4mm_P0.5mm_EP2.7x2.7mm, symbol QuadPreRecorder:TPA6130A2RTJ
- added U12: ADP7142AUJZ, Package_TO_SOT_SMD:TSOT-23-5, symbol Regulator_Linear:ADP7142AUJZ
- added U15, U4, U5: CD4053BPW, Package_SO:TSSOP-16_4.4x5mm_P0.65mm, symbol Analog_Switch:CD4053B
- added U16, U6: OPA1654, Package_SO:TSSOP-14_4.4x5mm_P0.65mm, symbol QuadPreRecorder:OPA1654
- added U7: PCM1864DBT, Package_SO:TSSOP-30_4.4x7.8mm_P0.5mm, symbol Audio:PCM1864DBT
- added U8: Teensy 4.1, QuadPreRecorder:Teensy41_Socket, symbol QuadPreRecorder:Teensy41
- added U9: PCM5102A, Package_SO:TSSOP-20_4.4x6.5mm_P0.65mm, symbol QuadPreRecorder:PCM5102A
- C1: renamed from U2; value TPS7A2033PDBV -> 100uF 25V; footprint Package_TO_SOT_SMD:SOT-23-5 -> Capacitor_SMD:CP_Elec_6.3x5.8; symbol QuadPreRecorder:TPS7A20DBV -> Device:C_Polarized; AltMPN (none) -> Lelon VZS101M1ETR-0606; LCSC (none) -> C178590; MPN TPS7A2033PDBVR -> EEE-FT1E101AP; Manufacturer Texas Instruments -> Panasonic
- C10: renamed from R11; value 100R RF -> 47uF 10V; footprint Resistor_SMD:R_0603_1608Metric -> Capacitor_SMD:C_1206_3216Metric; symbol Device:R -> Device:C; AltMPN (none) -> Murata GRM31CR61A476ME15K; LCSC (none) -> C385907; MPN RC0603FR series, 1% -> EMK316BBJ476ML-T; Manufacturer Yageo -> Taiyo Yuden
- C101: renamed from C46; value 10uF -> 4.7uF 35V FILM; footprint Capacitor_SMD:C_1206_3216Metric -> Capacitor_SMD:C_1812_4532Metric; AltMPN (none) -> Rubycon 16MU475MC14532; LCSC (none) -> C3778321; MPN GRM series X7R/C0G -> 35MU475KC44532; Manufacturer Murata -> Rubycon
- C102: renamed from J3; value MSP3520 TFT 3.5IN 14PIN HEADER -> 4.7uF 35V FILM; footprint Connector_PinHeader_2.54mm:PinHeader_1x14_P2.54mm_Vertical -> Capacitor_SMD:C_1812_4532Metric; symbol Connector_Generic:Conn_01x14 -> Device:C; AltMPN (none) -> Rubycon 16MU475MC14532; LCSC (none) -> C3778321; MPN PRPC014SAAN-RC -> 35MU475KC44532; Manufacturer Sullins Connector Solutions -> Rubycon
- C103: renamed from R63; value 470R -> 4.7uF 35V FILM; footprint Resistor_SMD:R_0603_1608Metric -> Capacitor_SMD:C_1812_4532Metric; symbol Device:R -> Device:C; AltMPN (none) -> Rubycon 16MU475MC14532; LCSC (none) -> C3778321; MPN RC0603FR series, 1% -> 35MU475KC44532; Manufacturer Yageo -> Rubycon
- C105: renamed from SW4; value TFT MENU NAV -> 22pF C0G; footprint QuadPreRecorder:SW_Nav_ALPS_SKQUCAA010 -> Capacitor_SMD:C_0603_1608Metric; symbol QuadPreRecorder:SW_Nav5 -> Device:C; AltMPN (none) -> FOJAN FCC0603N220J500CT; LCSC (none) -> C408549; MPN SKQUCAA010 -> GCM1885C2A220JA16D; Manufacturer Alps Alpine -> Murata
- C106: renamed from D5; value RECORD RED -> 22pF C0G; footprint LED_SMD:LED_0603_1608Metric -> Capacitor_SMD:C_0603_1608Metric; symbol Device:LED -> Device:C; AltMPN (none) -> FOJAN FCC0603N220J500CT; LCSC (none) -> C408549; MPN LTST-C190KRKT -> GCM1885C2A220JA16D; Manufacturer Lite-On -> Murata
- C107: renamed from C57; value 680nF X7R -> 22pF C0G; footprint Capacitor_SMD:C_0805_2012Metric -> Capacitor_SMD:C_0603_1608Metric; AltMPN (none) -> FOJAN FCC0603N220J500CT; LCSC (none) -> C408549; MPN GRM series X7R/C0G -> GCM1885C2A220JA16D
- C11: renamed from C14; value 100pF C0G -> 100nF; AltMPN (none) -> Yageo CC0603KRX7R9BB104; LCSC (none) -> C1591; MPN GRM series X7R/C0G -> CL10B104KB8NNNC; Manufacturer Murata -> Samsung
- C12: renamed from U6; value OPA1654 -> 1nF 1kV C0G; footprint Package_SO:TSSOP-14_4.4x5mm_P0.65mm -> Capacitor_SMD:C_0805_2012Metric; symbol QuadPreRecorder:OPA1654 -> Device:C; AltMPN (none) -> Murata GRM31C5C3A102JWA3L; LCSC (none) -> C309495; MPN OPA1654AIPWR -> CC0805KRX7RCBB102; Manufacturer Texas Instruments -> Yageo
- C13: renamed from C43; value 100nF -> 100pF C0G; AltMPN (none) -> Samsung CL10C101JB8NNNC; LCSC (none) -> C71664; MPN GRM series X7R/C0G -> GRM1885C1H101JA01D
- C14: renamed from R72; value 10k -> 100pF C0G; footprint Resistor_SMD:R_0603_1608Metric -> Capacitor_SMD:C_0603_1608Metric; symbol Device:R -> Device:C; AltMPN (none) -> Samsung CL10C101JB8NNNC; LCSC (none) -> C71664; MPN RC0603FR series, 1% -> GRM1885C1H101JA01D; Manufacturer Yageo -> Murata
- C15: renamed from U9; value PCM5102A -> 100pF C0G; footprint Package_SO:TSSOP-20_4.4x6.5mm_P0.65mm -> Capacitor_SMD:C_0603_1608Metric; symbol QuadPreRecorder:PCM5102A -> Device:C; AltMPN (none) -> Samsung CL10C101JB8NNNC; LCSC (none) -> C71664; MPN PCM5102APWR -> GRM1885C1H101JA01D; Manufacturer Texas Instruments -> Murata
- C16: renamed from C59; value 1uF -> 100pF C0G; AltMPN (none) -> Samsung CL10C101JB8NNNC; LCSC (none) -> C71664; MPN GRM series X7R/C0G -> GRM1885C1H101JA01D
- C17: renamed from C44; value 100nF -> 4.7uF 35V FILM; footprint Capacitor_SMD:C_0603_1608Metric -> Capacitor_SMD:C_1812_4532Metric; AltMPN (none) -> Rubycon 16MU475MC14532; LCSC (none) -> C3778321; MPN GRM series X7R/C0G -> 35MU475KC44532; Manufacturer Murata -> Rubycon
- C18: renamed from R73; value 10k -> 4.7uF 35V FILM; footprint Resistor_SMD:R_0603_1608Metric -> Capacitor_SMD:C_1812_4532Metric; symbol Device:R -> Device:C; AltMPN (none) -> Rubycon 16MU475MC14532; LCSC (none) -> C3778321; MPN RC0603FR series, 1% -> 35MU475KC44532; Manufacturer Yageo -> Rubycon
- C19: renamed from C51; value 2.2uF -> 4.7uF 35V FILM; footprint Capacitor_SMD:C_0805_2012Metric -> Capacitor_SMD:C_1812_4532Metric; AltMPN (none) -> Rubycon 16MU475MC14532; LCSC (none) -> C3778321; MPN GRM series X7R/C0G -> 35MU475KC44532; Manufacturer Murata -> Rubycon
- C2: renamed from D7; value PESD12VL1BA -> 100nF 25V; footprint Diode_SMD:D_SOD-323 -> Capacitor_SMD:C_0805_2012Metric; symbol Device:D_TVS -> Device:C; AltMPN (none) -> Yageo CC0805KRX7R9BB104; LCSC (none) -> C28233; MPN PESD12VL1BA,115 -> CL21B104KCFNNNE; Manufacturer Nexperia -> Samsung
- C20: renamed from C60; value 2.2uF -> 4.7uF 35V FILM; footprint Capacitor_SMD:C_0603_1608Metric -> Capacitor_SMD:C_1812_4532Metric; AltMPN (none) -> Rubycon 16MU475MC14532; LCSC (none) -> C3778321; MPN GRM series X7R/C0G -> 35MU475KC44532; Manufacturer Murata -> Rubycon
- C21: renamed from R46; value 33R -> 22pF C0G; footprint Resistor_SMD:R_0603_1608Metric -> Capacitor_SMD:C_0603_1608Metric; symbol Device:R -> Device:C; AltMPN (none) -> FOJAN FCC0603N220J500CT; LCSC (none) -> C408549; MPN RC0603FR series, 1% -> GCM1885C2A220JA16D; Manufacturer Yageo -> Murata
- C22: renamed from C73; value 100nF -> 22pF C0G; AltMPN (none) -> FOJAN FCC0603N220J500CT; LCSC (none) -> C408549; MPN GRM series X7R/C0G -> GCM1885C2A220JA16D
- C23: renamed from C64; value 100nF -> 22pF C0G; AltMPN (none) -> FOJAN FCC0603N220J500CT; LCSC (none) -> C408549; MPN GRM series X7R/C0G -> GCM1885C2A220JA16D
- C24: renamed from J5; value 1/8in BINAURAL HEADPHONE OUT -> 22pF C0G; footprint Connector_Audio:Jack_3.5mm_CUI_SJ1-3533NG_Horizontal -> Capacitor_SMD:C_0603_1608Metric; symbol Connector_Audio:AudioJack3 -> Device:C; AltMPN (none) -> FOJAN FCC0603N220J500CT; LCSC (none) -> C408549; MPN SJ1-3533NG -> GCM1885C2A220JA16D; Manufacturer CUI Devices -> Murata
- C25: renamed from R47; value 33R -> 4.7uF 35V FILM; footprint Resistor_SMD:R_0603_1608Metric -> Capacitor_SMD:C_1812_4532Metric; symbol Device:R -> Device:C; AltMPN (none) -> Rubycon 16MU475MC14532; LCSC (none) -> C3778321; MPN RC0603FR series, 1% -> 35MU475KC44532; Manufacturer Yageo -> Rubycon
- C26: renamed from R51; value 10k -> 4.7uF 35V FILM; footprint Resistor_SMD:R_0603_1608Metric -> Capacitor_SMD:C_1812_4532Metric; symbol Device:R -> Device:C; AltMPN (none) -> Rubycon 16MU475MC14532; LCSC (none) -> C3778321; MPN RC0603FR series, 1% -> 35MU475KC44532; Manufacturer Yageo -> Rubycon
- C27: renamed from R57; value 33R -> 4.7uF 35V FILM; footprint Resistor_SMD:R_0603_1608Metric -> Capacitor_SMD:C_1812_4532Metric; symbol Device:R -> Device:C; AltMPN (none) -> Rubycon 16MU475MC14532; LCSC (none) -> C3778321; MPN RC0603FR series, 1% -> 35MU475KC44532; Manufacturer Yageo -> Rubycon
- C29: renamed from R49; value 33R -> 10nF C0G; footprint Resistor_SMD:R_0603_1608Metric -> Capacitor_SMD:C_0603_1608Metric; symbol Device:R -> Device:C; AltMPN (none) -> Murata GRM1885C1H103JA01J; LCSC (none) -> C76599; MPN RC0603FR series, 1% -> C1608C0G1H103JT000N; Manufacturer Yageo -> TDK
- C3: renamed from D8; value PESD12VL1BA -> 10uF 25V; footprint Diode_SMD:D_SOD-323 -> Capacitor_SMD:C_1206_3216Metric; symbol Device:D_TVS -> Device:C; AltMPN (none) -> Murata GRM31CR71E106KA12L; LCSC (none) -> C14860; MPN PESD12VL1BA,115 -> CL31B106KAHNNNE; Manufacturer Nexperia -> Samsung
- C30: renamed from R53; value 10k -> 10nF C0G; footprint Resistor_SMD:R_0603_1608Metric -> Capacitor_SMD:C_0603_1608Metric; symbol Device:R -> Device:C; AltMPN (none) -> Murata GRM1885C1H103JA01J; LCSC (none) -> C76599; MPN RC0603FR series, 1% -> C1608C0G1H103JT000N; Manufacturer Yageo -> TDK
- C31: renamed from R59; value 33R -> 10nF C0G; footprint Resistor_SMD:R_0603_1608Metric -> Capacitor_SMD:C_0603_1608Metric; symbol Device:R -> Device:C; AltMPN (none) -> Murata GRM1885C1H103JA01J; LCSC (none) -> C76599; MPN RC0603FR series, 1% -> C1608C0G1H103JT000N; Manufacturer Yageo -> TDK
- C4: renamed from C17; value 4.7uF 16V -> 22pF C0G; footprint Capacitor_SMD:C_1206_3216Metric -> Capacitor_SMD:C_0603_1608Metric; AltMPN (none) -> FOJAN FCC0603N220J500CT; LCSC (none) -> C408549; MPN GRM series X7R/C0G -> GCM1885C2A220JA16D
- C5: renamed from R14; value 1M -> 22uF 10V; footprint Resistor_SMD:R_0603_1608Metric -> Capacitor_SMD:C_1206_3216Metric; symbol Device:R -> Device:C; AltMPN (none) -> Murata GRM31CZ71C226ME15L; LCSC (none) -> C385906; MPN RC0603FR series, 1% -> EMK316BB7226ML-T; Manufacturer Yageo -> Taiyo Yuden
- C6: renamed from R18; value 68k 0.1% -> 22uF 10V; footprint Resistor_SMD:R_0603_1608Metric -> Capacitor_SMD:C_1206_3216Metric; symbol Device:R -> Device:C; AltMPN (none) -> Murata GRM31CZ71C226ME15L; LCSC (none) -> C385906; MPN TNPW0603 series, 0.1% -> EMK316BB7226ML-T; Manufacturer Vishay -> Taiyo Yuden
- C66: renamed from C15; value 100pF C0G -> 100uF 16V; footprint Capacitor_SMD:C_0603_1608Metric -> Capacitor_SMD:CP_Elec_6.3x5.8; symbol Device:C -> Device:C_Polarized; AltMPN (none) -> Lelon VZL101M1CTR-0606; LCSC (none) -> C128532; MPN GRM series X7R/C0G -> EEE-FK1C101P; Manufacturer Murata -> Panasonic
- C7: renamed from R30; value 90.9k 0.1% -> 1uF 10V; footprint Resistor_SMD:R_0603_1608Metric -> Capacitor_SMD:C_0805_2012Metric; symbol Device:R -> Device:C; AltMPN (none) -> Samsung CL21B105KBFNNNE; LCSC (none) -> C91185; MPN TNPW0603 series, 0.1% -> CC0805KKX7R9BB105; Manufacturer Vishay -> Yageo
- C74: renamed from C12; value 1nF 1kV C0G -> 10uF 16V; footprint Capacitor_SMD:C_0805_2012Metric -> Capacitor_SMD:C_1206_3216Metric; AltMPN (none) -> Murata GRM31CR71E106KA12L; LCSC (none) -> C14860; MPN GRM series X7R/C0G -> CL31B106KAHNNNE; Manufacturer Murata -> Samsung
- C75: renamed from D6; value PESD12VL1BA -> 100nF; footprint Diode_SMD:D_SOD-323 -> Capacitor_SMD:C_0603_1608Metric; symbol Device:D_TVS -> Device:C; AltMPN (none) -> Yageo CC0603KRX7R9BB104; LCSC (none) -> C1591; MPN PESD12VL1BA,115 -> CL10B104KB8NNNC; Manufacturer Nexperia -> Samsung
- C76: renamed from C10; value 47uF 10V -> 10uF 25V; AltMPN (none) -> Murata GRM31CR71E106KA12L; LCSC (none) -> C14860; MPN GRM series X7R/C0G -> CL31B106KAHNNNE; Manufacturer Murata -> Samsung
- C77: renamed from C11; value 100nF -> 10uF 25V; footprint Capacitor_SMD:C_0603_1608Metric -> Capacitor_SMD:C_1206_3216Metric; AltMPN (none) -> Murata GRM31CR71E106KA12L; LCSC (none) -> C14860; MPN GRM series X7R/C0G -> CL31B106KAHNNNE; Manufacturer Murata -> Samsung
- C78: renamed from C6; value 22uF 10V -> 100nF; footprint Capacitor_SMD:C_1206_3216Metric -> Capacitor_SMD:C_0603_1608Metric; AltMPN (none) -> Yageo CC0603KRX7R9BB104; LCSC (none) -> C1591; MPN GRM series X7R/C0G -> CL10B104KB8NNNC; Manufacturer Murata -> Samsung
- C8: renamed from C21; value 22pF C0G -> 4.7uF 10V; footprint Capacitor_SMD:C_0603_1608Metric -> Capacitor_SMD:C_0805_2012Metric; AltMPN (none) -> Samsung CL21B475KAFNNNE; LCSC (none) -> C437556; MPN GRM series X7R/C0G -> GRM21BZ71E475KE15L
- C83: renamed from R4; value 1M -> 2.2uF; footprint Resistor_SMD:R_0603_1608Metric -> Capacitor_SMD:C_0805_2012Metric; symbol Device:R -> Device:C; AltMPN (none) -> Murata GRM21BR71E225KE11K; LCSC (none) -> C19110; MPN RC0603FR series, 1% -> CL21B225KAFNNNE; Manufacturer Yageo -> Samsung
- C85: renamed from C7; value 1uF 10V -> 10uF 25V; footprint Capacitor_SMD:C_0805_2012Metric -> Capacitor_SMD:C_1206_3216Metric; AltMPN (none) -> Murata GRM31CR71E106KA12L; LCSC (none) -> C14860; MPN GRM series X7R/C0G -> CL31B106KAHNNNE; Manufacturer Murata -> Samsung
- C88: renamed from R5; value 0R CHASSIS LINK -> 10uF 16V; footprint Resistor_SMD:R_0603_1608Metric -> Capacitor_SMD:C_1206_3216Metric; symbol Device:R -> Device:C; AltMPN (none) -> Murata GRM31CR71E106KA12L; LCSC (none) -> C14860; MPN RC0603FR series, 1% -> CL31B106KAHNNNE; Manufacturer Yageo -> Samsung; now fitted
- C89: renamed from R37; value 100R -> 100nF; footprint Resistor_SMD:R_0603_1608Metric -> Capacitor_SMD:C_0603_1608Metric; symbol Device:R -> Device:C; AltMPN (none) -> Yageo CC0603KRX7R9BB104; LCSC (none) -> C1591; MPN RC0603FR series, 1% -> CL10B104KB8NNNC; Manufacturer Yageo -> Samsung
- C9: renamed from R7; value 4.7k ELECTRET BIAS -> 1uF 10V; footprint Resistor_SMD:R_0603_1608Metric -> Capacitor_SMD:C_0805_2012Metric; symbol Device:R -> Device:C; AltMPN (none) -> Samsung CL21B105KBFNNNE; LCSC (none) -> C91185; MPN RC0603FR series, 1% -> CC0805KKX7R9BB105
- C90: renamed from R40; value 100k -> 10uF 10V; footprint Resistor_SMD:R_0603_1608Metric -> Capacitor_SMD:C_0805_2012Metric; symbol Device:R -> Device:C; AltMPN (none) -> Samsung CL21B106KOQNNNE; LCSC (none) -> C237493; MPN RC0603FR series, 1% -> GRM21BZ71E106KE15L; Manufacturer Yageo -> Murata; now fitted
- C91: renamed from R9; value 4.7k ELECTRET BIAS -> 10uF 10V; footprint Resistor_SMD:R_0603_1608Metric -> Capacitor_SMD:C_0805_2012Metric; symbol Device:R -> Device:C; AltMPN (none) -> Samsung CL21B106KOQNNNE; LCSC (none) -> C237493; MPN RC0603FR series, 1% -> GRM21BZ71E106KE15L; Manufacturer Yageo -> Murata
- C92: renamed from R13; value 100R RF -> 10uF 10V; footprint Resistor_SMD:R_0603_1608Metric -> Capacitor_SMD:C_0805_2012Metric; symbol Device:R -> Device:C; AltMPN (none) -> Samsung CL21B106KOQNNNE; LCSC (none) -> C237493; MPN RC0603FR series, 1% -> GRM21BZ71E106KE15L; Manufacturer Yageo -> Murata
- C95: renamed from R34; value 100R -> 1uF 10V; footprint Resistor_SMD:R_0603_1608Metric -> Capacitor_SMD:C_0805_2012Metric; symbol Device:R -> Device:C; AltMPN (none) -> Samsung CL21B105KBFNNNE; LCSC (none) -> C91185; MPN RC0603FR series, 1% -> CC0805KKX7R9BB105
- C96: renamed from C29; value 10nF C0G -> 4.7uF 10V; footprint Capacitor_SMD:C_0603_1608Metric -> Capacitor_SMD:C_0805_2012Metric; AltMPN (none) -> Samsung CL21B475KAFNNNE; LCSC (none) -> C437556; MPN GRM series X7R/C0G -> GRM21BZ71E475KE15L
- C97: renamed from D3; value SS14 -> 100pF C0G; footprint Diode_SMD:D_SMA -> Capacitor_SMD:C_0603_1608Metric; symbol Device:D_Schottky -> Device:C; AltMPN (none) -> Samsung CL10C101JB8NNNC; LCSC (none) -> C71664; MPN SS14-13-F -> GRM1885C1H101JA01D; Manufacturer Diodes Incorporated -> Murata
- C98: renamed from C50; value 100nF -> 100pF C0G; AltMPN (none) -> Samsung CL10C101JB8NNNC; LCSC (none) -> C71664; MPN GRM series X7R/C0G -> GRM1885C1H101JA01D
- C99: renamed from R62; value 470R -> 100pF C0G; footprint Resistor_SMD:R_0603_1608Metric -> Capacitor_SMD:C_0603_1608Metric; symbol Device:R -> Device:C; AltMPN (none) -> Samsung CL10C101JB8NNNC; LCSC (none) -> C71664; MPN RC0603FR series, 1% -> GRM1885C1H101JA01D; Manufacturer Yageo -> Murata
- D1: value SS14 -> B340A 40V 3A; AltMPN (none) -> LangJie SS34 SMA; LCSC (none) -> C7450457; MPN SS14-13-F -> B340A-13-F
- D10: renamed from R2; value 130k -> B340A 40V 3A; footprint Resistor_SMD:R_0603_1608Metric -> Diode_SMD:D_SMA; symbol Device:R -> Device:D_Schottky; AltMPN (none) -> LangJie SS34 SMA; LCSC (none) -> C7450457; MPN RC0603FR series, 1% -> B340A-13-F; Manufacturer Yageo -> Diodes Incorporated
- D11: renamed from C3; value 10uF 25V -> USBLC6-2SC6; footprint Capacitor_SMD:C_1206_3216Metric -> Package_TO_SOT_SMD:SOT-23-6; symbol Device:C -> Power_Protection:USBLC6-2P6; MPN GRM series X7R/C0G -> USBLC6-2SC6; Manufacturer Murata -> STMicroelectronics
- D12: renamed from C9; value 1uF 10V -> B340A 40V 3A; footprint Capacitor_SMD:C_0805_2012Metric -> Diode_SMD:D_SMA; symbol Device:C -> Device:D_Schottky; AltMPN (none) -> LangJie SS34 SMA; LCSC (none) -> C7450457; MPN GRM series X7R/C0G -> B340A-13-F; Manufacturer Murata -> Diodes Incorporated
- D14: renamed from R29; value 10k 0.1% -> B340A 40V 3A; footprint Resistor_SMD:R_0603_1608Metric -> Diode_SMD:D_SMA; symbol Device:R -> Device:D_Schottky; AltMPN (none) -> LangJie SS34 SMA; LCSC (none) -> C7450457; MPN TNPW0603 series, 0.1% -> B340A-13-F; Manufacturer Vishay -> Diodes Incorporated
- D15: renamed from R42; value 100k -> 1N4148W; footprint Resistor_SMD:R_0603_1608Metric -> Diode_SMD:D_SOD-123; symbol Device:R -> Device:D_Schottky; AltMPN (none) -> ST(Semtech) 1N4148W; LCSC (none) -> C81598; MPN RC0603FR series, 1% -> 1N4148W-7-F; Manufacturer Yageo -> Diodes Incorporated
- D16: renamed from R43; value 47k -> 1N4148W; footprint Resistor_SMD:R_0603_1608Metric -> Diode_SMD:D_SOD-123; symbol Device:R -> Device:D_Schottky; AltMPN (none) -> ST(Semtech) 1N4148W; LCSC (none) -> C81598; MPN RC0603FR series, 1% -> 1N4148W-7-F; Manufacturer Yageo -> Diodes Incorporated
- D17: renamed from R68; value 1k -> 1N4148W; footprint Resistor_SMD:R_0603_1608Metric -> Diode_SMD:D_SOD-123; symbol Device:R -> Device:D_Schottky; AltMPN (none) -> ST(Semtech) 1N4148W; LCSC (none) -> C81598; MPN RC0603FR series, 1% -> 1N4148W-7-F; Manufacturer Yageo -> Diodes Incorporated
- D18: renamed from C33; value 100nF -> 1N4148W; footprint Capacitor_SMD:C_0603_1608Metric -> Diode_SMD:D_SOD-123; symbol Device:C -> Device:D_Schottky; AltMPN (none) -> ST(Semtech) 1N4148W; LCSC (none) -> C81598; MPN GRM series X7R/C0G -> 1N4148W-7-F; Manufacturer Murata -> Diodes Incorporated
- D19: renamed from C34; value 100nF -> 1N4148W; footprint Capacitor_SMD:C_0603_1608Metric -> Diode_SMD:D_SOD-123; symbol Device:C -> Device:D_Schottky; AltMPN (none) -> ST(Semtech) 1N4148W; LCSC (none) -> C81598; MPN GRM series X7R/C0G -> 1N4148W-7-F; Manufacturer Murata -> Diodes Incorporated
- D2: renamed from R3; value 100k -> SMBJ12A; footprint Resistor_SMD:R_0603_1608Metric -> Diode_SMD:D_SMB; symbol Device:R -> Device:D_TVS; MPN RC0603FR series, 1% -> SMBJ12A; Manufacturer Yageo -> Littelfuse
- D20: renamed from U7; value PCM1864DBT -> PESD12VL1BA; footprint Package_SO:TSSOP-30_4.4x7.8mm_P0.5mm -> Diode_SMD:D_SOD-323; symbol Audio:PCM1864DBT -> Device:D_TVS; MPN PCM1864DBTR -> PESD12VL1BA,115; Manufacturer Texas Instruments -> Nexperia
- D21: renamed from C38; value 1uF -> PESD12VL1BA; footprint Capacitor_SMD:C_0805_2012Metric -> Diode_SMD:D_SOD-323; symbol Device:C -> Device:D_TVS; MPN GRM series X7R/C0G -> PESD12VL1BA,115; Manufacturer Murata -> Nexperia
- D22: renamed from C39; value 1uF -> PESD12VL1BA; footprint Capacitor_SMD:C_0805_2012Metric -> Diode_SMD:D_SOD-323; symbol Device:C -> Device:D_TVS; MPN GRM series X7R/C0G -> PESD12VL1BA,115; Manufacturer Murata -> Nexperia
- D23: renamed from C40; value 100nF -> PESD12VL1BA; footprint Capacitor_SMD:C_0603_1608Metric -> Diode_SMD:D_SOD-323; symbol Device:C -> Device:D_TVS; MPN GRM series X7R/C0G -> PESD12VL1BA,115; Manufacturer Murata -> Nexperia
- D24: renamed from R39; value 100k -> BAT54; footprint Resistor_SMD:R_0603_1608Metric -> Diode_SMD:D_SOD-123; symbol Device:R -> Device:D_Small; MPN RC0603FR series, 1% -> BAT54-7-F; Manufacturer Yageo -> Diodes Incorporated; now fitted
- D6, D7: renamed from U6; value OPA1654 -> PESD12VL1BA; footprint Package_SO:TSSOP-14_4.4x5mm_P0.65mm -> Diode_SMD:D_SOD-323; symbol QuadPreRecorder:OPA1654 -> Device:D_TVS; MPN OPA1654AIPWR -> PESD12VL1BA,115; Manufacturer Texas Instruments -> Nexperia
- D8: renamed from C36; value 100nF -> PESD12VL1BA; footprint Capacitor_SMD:C_0603_1608Metric -> Diode_SMD:D_SOD-323; symbol Device:C -> Device:D_TVS; MPN GRM series X7R/C0G -> PESD12VL1BA,115; Manufacturer Murata -> Nexperia
- D9: renamed from C37; value 10uF 16V -> PESD12VL1BA; footprint Capacitor_SMD:C_1206_3216Metric -> Diode_SMD:D_SOD-323; symbol Device:C -> Device:D_TVS; MPN GRM series X7R/C0G -> PESD12VL1BA,115; Manufacturer Murata -> Nexperia
- F2: renamed from R1; value 680k -> 2A PTC; footprint Resistor_SMD:R_0603_1608Metric -> Fuse:Fuse_1206_3216Metric; symbol Device:R -> Device:Polyfuse; MPN RC0603FR series, 1% -> 1206L200PR; Manufacturer Yageo -> Littelfuse
- J10: renamed from R33; value 90.9k 0.1% -> BATTERY 1S LiPo; footprint Resistor_SMD:R_0603_1608Metric -> Connector_JST:JST_PH_B2B-PH-K_1x02_P2.00mm_Vertical; symbol Device:R -> Connector_Generic:Conn_01x02; MPN TNPW0603 series, 0.1% -> B2B-PH-K-S; Manufacturer Vishay -> JST
- J2: renamed from C35; value 100nF -> AMBISONIC MIC RJ45; footprint Capacitor_SMD:C_0603_1608Metric -> Connector_RJ:RJ45_Amphenol_RJHSE5380; symbol Device:C -> Connector:8P8C_Shielded; MPN GRM series X7R/C0G -> RJHSE-5380; Manufacturer Murata -> Amphenol ICC
- J9: renamed from D2; value SMBJ12A -> USB-C POWER + DATA; footprint Diode_SMD:D_SMB -> Connector_USB:USB_C_Receptacle_HRO_TYPE-C-31-M-12; symbol Device:D_TVS -> Connector:USB_C_Receptacle_USB2.0_16P; MPN SMBJ12A -> TYPE-C-31-M-12; Manufacturer Littelfuse -> HRO
- L1: renamed from R6; value 4.7k ELECTRET BIAS -> 2.2uH 1.5A; footprint Resistor_SMD:R_0603_1608Metric -> Inductor_SMD:L_Abracon_ASPIAIG-F4020; symbol Device:R -> Device:L; MPN RC0603FR series, 1% -> ASPIAIG-F4020-2R2M-T; Manufacturer Yageo -> Abracon
- L2: renamed from U3; value TLE2426ID -> 10uH 2A; footprint Package_SO:SOIC-8_3.9x4.9mm_P1.27mm -> Inductor_SMD:L_Bourns_SRN6045TA; symbol Reference_Voltage:TLE2426xD -> Device:L; MPN TLE2426IDR -> SRN6045TA-100M; Manufacturer Texas Instruments -> Bourns
- Q3: renamed from C32; value 10nF C0G -> AO3401A; footprint Capacitor_SMD:C_0603_1608Metric -> Package_TO_SOT_SMD:SOT-23; symbol Device:C -> Transistor_FET:Q_PMOS_GSD; MPN GRM series X7R/C0G -> AO3401A; Manufacturer Murata -> Alpha & Omega
- Q4: renamed from R41; value 100k -> AO3401A; footprint Resistor_SMD:R_0603_1608Metric -> Package_TO_SOT_SMD:SOT-23; symbol Device:R -> Transistor_FET:Q_PMOS_GSD; MPN RC0603FR series, 1% -> AO3401A; Manufacturer Yageo -> Alpha & Omega; now fitted
- Q6: renamed from C18; value 4.7uF 16V -> AO3401A; footprint Capacitor_SMD:C_1206_3216Metric -> Package_TO_SOT_SMD:SOT-23; symbol Device:C -> Transistor_FET:Q_PMOS_GSD; MPN GRM series X7R/C0G -> AO3401A; Manufacturer Murata -> Alpha & Omega
- Q7: renamed from R20; value 68k 0.1% -> 2N7002; footprint Resistor_SMD:R_0603_1608Metric -> Package_TO_SOT_SMD:SOT-23; symbol Device:R -> Transistor_FET:Q_NMOS_GSD; MPN TNPW0603 series, 0.1% -> 2N7002NXAKR; Manufacturer Vishay -> Nexperia
- Q8: renamed from R31; value 90.9k 0.1% -> AO3401A; footprint Resistor_SMD:R_0603_1608Metric -> Package_TO_SOT_SMD:SOT-23; symbol Device:R -> Transistor_FET:Q_PMOS_GSD; MPN TNPW0603 series, 0.1% -> AO3401A; Manufacturer Vishay -> Alpha & Omega
- Q9: renamed from C26; value 4.7uF 16V -> 2N7002; footprint Capacitor_SMD:C_1206_3216Metric -> Package_TO_SOT_SMD:SOT-23; symbol Device:C -> Transistor_FET:Q_NMOS_GSD; MPN GRM series X7R/C0G -> 2N7002NXAKR; Manufacturer Murata -> Nexperia
- R1: renamed from R10; value 100R RF -> 680k; AltMPN (none) -> UNI-ROYAL 0603WAF6803T5E; LCSC (none) -> C25822; MPN RC0603FR series, 1% -> RC0603FR-07680KL
- R10: renamed from C42; value 10uF -> 100R RF; footprint Capacitor_SMD:C_1206_3216Metric -> Resistor_SMD:R_0603_1608Metric; symbol Device:C -> Device:R; AltMPN (none) -> UNI-ROYAL 0603WAF1000T5E; LCSC (none) -> C22775; MPN GRM series X7R/C0G -> RC0603FR-07100RL; Manufacturer Murata -> Yageo
- R100: renamed from R27; value 10k 0.1% -> 100k; AltMPN (none) -> UNI-ROYAL 0603WAF1003T5E; LCSC (none) -> C25803; MPN TNPW0603 series, 0.1% -> RC0603FR-07100KL; Manufacturer Vishay -> Yageo
- R101: renamed from C22; value 22pF C0G -> 100k; footprint Capacitor_SMD:C_0603_1608Metric -> Resistor_SMD:R_0603_1608Metric; symbol Device:C -> Device:R; AltMPN (none) -> UNI-ROYAL 0603WAF1003T5E; LCSC (none) -> C25803; MPN GRM series X7R/C0G -> RC0603FR-07100KL; Manufacturer Murata -> Yageo
- R102: renamed from R35; AltMPN (none) -> UNI-ROYAL 0603WAF1000T5E; LCSC (none) -> C22775; MPN RC0603FR series, 1% -> RC0603FR-07100RL
- R103: renamed from C30; value 10nF C0G -> 100k; footprint Capacitor_SMD:C_0603_1608Metric -> Resistor_SMD:R_0603_1608Metric; symbol Device:C -> Device:R; AltMPN (none) -> UNI-ROYAL 0603WAF1003T5E; LCSC (none) -> C25803; MPN GRM series X7R/C0G -> RC0603FR-07100KL; Manufacturer Murata -> Yageo
- R104: renamed from R8; value 4.7k ELECTRET BIAS -> 100k BLEED; AltMPN (none) -> UNI-ROYAL 0603WAF1003T5E; LCSC (none) -> C25803; MPN RC0603FR series, 1% -> RC0603FR-07100KL
- R11: renamed from R71; value 10k -> 100R RF; AltMPN (none) -> UNI-ROYAL 0603WAF1000T5E; LCSC (none) -> C22775; MPN RC0603FR series, 1% -> RC0603FR-07100RL
- R110: renamed from U8; value Teensy 4.1 -> 100R RF; footprint QuadPreRecorder:Teensy41_Socket -> Resistor_SMD:R_0603_1608Metric; symbol QuadPreRecorder:Teensy41 -> Device:R; AltMPN (none) -> UNI-ROYAL 0603WAF1000T5E; LCSC (none) -> C22775; MPN TEENSY41 -> RC0603FR-07100RL; Manufacturer PJRC -> Yageo
- R111: renamed from C49; value 10nF -> 100R RF; footprint Capacitor_SMD:C_0603_1608Metric -> Resistor_SMD:R_0603_1608Metric; symbol Device:C -> Device:R; AltMPN (none) -> UNI-ROYAL 0603WAF1000T5E; LCSC (none) -> C22775; MPN GRM series X7R/C0G -> RC0603FR-07100RL; Manufacturer Murata -> Yageo
- R112: renamed from R61; value 100R -> 100R RF; AltMPN (none) -> UNI-ROYAL 0603WAF1000T5E; LCSC (none) -> C22775; MPN RC0603FR series, 1% -> RC0603FR-07100RL
- R114: renamed from SW2; value RECORD START/STOP -> 1M; footprint Button_Switch_THT:SW_PUSH-12mm -> Resistor_SMD:R_0603_1608Metric; symbol Switch:SW_Push -> Device:R; AltMPN (none) -> UNI-ROYAL 0603WAF1004T5E; LCSC (none) -> C22935; MPN B3F-5150 -> RC0603FR-071ML; Manufacturer Omron -> Yageo
- R115: renamed from J6; value ANALOG TEST HEADER 2x13 -> 1M; footprint Connector_PinHeader_2.54mm:PinHeader_2x13_P2.54mm_Vertical -> Resistor_SMD:R_0603_1608Metric; symbol Connector_Generic:Conn_01x25 -> Device:R; AltMPN (none) -> UNI-ROYAL 0603WAF1004T5E; LCSC (none) -> C22935; MPN 2x13 0.1in pin header -> RC0603FR-071ML; Manufacturer Generic -> Yageo
- R116: renamed from C67; value 2.2nF C0G -> 1M; footprint Capacitor_SMD:C_0603_1608Metric -> Resistor_SMD:R_0603_1608Metric; symbol Device:C -> Device:R; AltMPN (none) -> UNI-ROYAL 0603WAF1004T5E; LCSC (none) -> C22935; MPN GRM series X7R/C0G -> RC0603FR-071ML; Manufacturer Murata -> Yageo
- R118: renamed from R50; value 10k -> 10k 0.1%; AltMPN (none) -> Vishay TNPW060310K0BEEA; LCSC (none) -> C95204; MPN RC0603FR series, 1% -> RT0603BRD0710KL
- R119: renamed from J7; value DIGITAL TEST HEADER 2x13 -> 10k 0.1%; footprint Connector_PinHeader_2.54mm:PinHeader_2x13_P2.54mm_Vertical -> Resistor_SMD:R_0603_1608Metric; symbol Connector_Generic:Conn_01x25 -> Device:R; AltMPN (none) -> Vishay TNPW060310K0BEEA; LCSC (none) -> C95204; MPN 2x13 0.1in pin header -> RT0603BRD0710KL; Manufacturer Generic -> Yageo
- R12: renamed from R56; value 100R TFT BACKLIGHT -> 100R RF; footprint Resistor_SMD:R_0805_2012Metric -> Resistor_SMD:R_0603_1608Metric; AltMPN (none) -> UNI-ROYAL 0603WAF1000T5E; LCSC (none) -> C22775; MPN RC0805FR-07100RL -> RC0603FR-07100RL
- R120: renamed from C68; value 2.2nF C0G -> 10k 0.1%; footprint Capacitor_SMD:C_0603_1608Metric -> Resistor_SMD:R_0603_1608Metric; symbol Device:C -> Device:R; AltMPN (none) -> Vishay TNPW060310K0BEEA; LCSC (none) -> C95204; MPN GRM series X7R/C0G -> RT0603BRD0710KL; Manufacturer Murata -> Yageo
- R122: renamed from C47; value 100nF -> 90.9k 0.1%; footprint Capacitor_SMD:C_0603_1608Metric -> Resistor_SMD:R_0603_1608Metric; symbol Device:C -> Device:R; AltMPN (none) -> Vishay TNPW060390K9BEEA; LCSC (none) -> C728600; MPN GRM series X7R/C0G -> RT0603BRD0790K9L; Manufacturer Murata -> Yageo
- R123: renamed from D4; value POWER BLUE -> 90.9k 0.1%; footprint LED_SMD:LED_0603_1608Metric -> Resistor_SMD:R_0603_1608Metric; symbol Device:LED -> Device:R; AltMPN (none) -> Vishay TNPW060390K9BEEA; LCSC (none) -> C728600; MPN LTST-C190TBKT -> RT0603BRD0790K9L; Manufacturer Lite-On -> Yageo
- R124: renamed from J4; value 1/4in BINAURAL LINE OUT -> 90.9k 0.1%; footprint Connector_Audio:Jack_6.35mm_Neutrik_NRJ6HF_Horizontal -> Resistor_SMD:R_0603_1608Metric; symbol Connector_Audio:AudioJack3 -> Device:R; AltMPN (none) -> Vishay TNPW060390K9BEEA; LCSC (none) -> C728600; MPN NRJ6HF -> RT0603BRD0790K9L; Manufacturer Neutrik -> Yageo
- R126: renamed from SW3; value MASTER GAIN -> 100k; footprint Rotary_Encoder:RotaryEncoder_Alps_EC11E-Switch_Vertical_H20mm -> Resistor_SMD:R_0603_1608Metric; symbol Device:RotaryEncoder_Switch -> Device:R; AltMPN (none) -> UNI-ROYAL 0603WAF1003T5E; LCSC (none) -> C25803; MPN EC11E15244G1 -> RC0603FR-07100KL; Manufacturer Alps Alpine -> Yageo
- R127: renamed from R54; value 2.2k -> 100k; AltMPN (none) -> UNI-ROYAL 0603WAF1003T5E; LCSC (none) -> C25803; MPN RC0603FR series, 1% -> RC0603FR-07100KL
- R128: renamed from RV1; value 10kA HEADPHONE VOLUME -> 100k; footprint QuadPreRecorder:RK097_Dual_Horizontal_NoEdgeGuide -> Resistor_SMD:R_0603_1608Metric; symbol Device:R_Potentiometer_Dual -> Device:R; AltMPN (none) -> UNI-ROYAL 0603WAF1003T5E; LCSC (none) -> C25803; MPN RK0971221-F15-C0-A103 -> RC0603FR-07100KL; Manufacturer Alps Alpine -> Yageo
- R13: renamed from U10; value TPA6132A2 -> 100R RF; footprint Package_DFN_QFN:WQFN-16-1EP_3x3mm_P0.5mm_EP1.6x1.6mm -> Resistor_SMD:R_0603_1608Metric; symbol Amplifier_Audio:TPA6132A2RTE -> Device:R; AltMPN (none) -> UNI-ROYAL 0603WAF1000T5E; LCSC (none) -> C22775; MPN TPA6132A2RTER -> RC0603FR-07100RL; Manufacturer Texas Instruments -> Yageo
- R131: renamed from J2; value AMBISONIC MIC RJ45 -> 20k; footprint Connector_RJ:RJ45_Amphenol_RJHSE5380 -> Resistor_SMD:R_0603_1608Metric; symbol Connector:8P8C_Shielded -> Device:R; AltMPN (none) -> UNI-ROYAL 0603WAF2002T5E; LCSC (none) -> C4184; MPN RJHSE-5380 -> RC0603FR-0720KL; Manufacturer Amphenol ICC -> Yageo
- R14: renamed from C45; value 10uF -> 1M; footprint Capacitor_SMD:C_1206_3216Metric -> Resistor_SMD:R_0603_1608Metric; symbol Device:C -> Device:R; AltMPN (none) -> UNI-ROYAL 0603WAF1004T5E; LCSC (none) -> C22935; MPN GRM series X7R/C0G -> RC0603FR-071ML; Manufacturer Murata -> Yageo
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Connections:
- net +3V3_A: now also C8.1, U2.5 (OUT), C41.1, C42.1, C54.1, C55.1, C64.1, U7.8 (AVDD), U9.1 (CPVDD), U9.8 (AVDD); no longer C1.5 (OUT), C15.1 (CPVDD), C15.8 (AVDD), C23.1, D20.8 (AVDD), R10.1, R23.1, R28.1, R6.1, U11.1
- net +3V3_D: now also R94.1, R95.1, R44.1, R45.1, R50.1, R51.1, R52.1, R53.1, R70.1, R71.1, R72.1, R73.1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; no longer C14.1, C15.20 (DVDD), C17.1, C18.1, C26.1, C30.1, D20.13 (DVDD), D20.14 (IOVDD), R11.1, R110.3V3A (3V3), R110.3V3B (3V3), R118.1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
- net +5V: now also C4.1, C5.1, C6.1, C7.1, C95.1, L1.2, Q8.2 (S), R1.1, R101.1, R3.1, U1.6 (VOS), U14.1 (IN)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; no longer C1.1 (IN), C1.3 (EN), C102.1 (Pin_1), C78.1, C85.1, C97.2 (A), D2.1, F2.1, R119.2 (Pin_2), R12.1, R127.1, R13.14 (VDD)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
- net +9V: now also C74.1, C75.1, C88.1, Q6.2 (S), R98.1, U3.3 (IN), C109.1, C110.1, C34.1, C35.1, C36.1, C37.1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; no longer D1.1 (K), D11.1, D19.1, D7.4 (V+), D8.1, D9.1, J2.1, J9.1 (A1), L2.3 (IN), R115.3 (Pin_3), R75.1, R76.1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
- net +9V_FUSED: now also D17.2 (A)
- net +9V_MIC: now also C66.1, R6.1, R67.2, R7.1, R8.1, R9.1; no longer C9.1, C91.1, L1.1, R80.2, R81.1
- net ADC_BCLK: now also R48.1, TP4.1, U8.21 (D21/BCLK1); no longer R110.21 (D21/BCLK1), R119.5 (Pin_5), R34.1
- net ADC_BCLK_IC: now also R48.2, U7.17 (BCK); no longer D20.17 (BCK), R34.2
- net ADC_DOUT2: now also R69.2, TP7.1, U8.6 (D6); no longer R110.6 (D6), R38.2
- net ADC_DOUT2_IC: now also R69.1, U7.22 (MISO/GPIO0/DMIN2); no longer D20.22 (MISO/GPIO0/DMIN2), R38.1
- net ADC_LDO: now also C43.1, C62.1, U7.11 (LDO); no longer C13.1, D20.11 (LDO), R18.1
- net ADC_LRCLK: now also R47.1, TP5.1, U8.20 (D20/LRCLK1); no longer C25.1, R110.20 (D20/LRCLK1), R119.6 (Pin_6)
- net ADC_LRCLK_IC: now also R47.2, U7.16 (LRCK); no longer C25.2, D20.16 (LRCK)
- net ADC_MCLK: now also R46.1, TP3.1, U8.23 (D23/MCLK1); no longer C21.1, R110.23 (D23/MCLK1), R119.4 (Pin_4)
- net ADC_MCLK_IC: now also R46.2, U7.15 (SCKI); no longer C21.2, D20.15 (SCKI)
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Other:
- note added: "192 kHz / 24-bit capture • real-time binaural monitor • two-layer Rev C (Hammond 1590XX, USB-C)"
- note added: "1S LiPo 5000 mAh on J10 (bottom). BQ24074 charges from USB only (0.74 A); the barrel and the boost bypass it. Hold RECORD + encoder push 2 s to power on/off on battery; USB or 9 V power the unit automatically."
- note added: "BATTERY + SOFT POWER (Rev C)"
- note added: "DISPLAY NOTE: J3 targets LCDWiki MSP3526 ST7796U + FT6336U 3.5in CAPACITIVE touch (480x320); module 98.0 x 55.5, holes 92.0 x 49.5 (LCDWiki spec V1.0) - verify against the physical module before drilling."
- note added: "PAD is a screen/firmware control (Rev C): Q1 drives four CD4053 paths, PAD_SELECT HIGH=direct, LOW=-9.7 dB. OPA1654 fixed gain is 20.1 dB."
- note added: "PCM5102A ground-centered line output through relay K1 (muted only while a USB host is attached); headphones = TPA6130A2 I2C-volume DirectPath amp fed from LINE_L/R (HP_ENABLE = /SD)."
- note added: "POWER: 9 V barrel / USB-C 5 V / 1S LiPo (BQ24074 charger, USB only) -> TPS61175 boost 10.45 V -> ADP7142 LDO 9 V analog rail; 5 V buck; 3.3 V audio LDO. Soft power: hold RECORD + encoder push 2 s (Q3/Q4 latch, KEEP_ON)."
- note added: "Rev C (2026-09-08) by jdg511 • https://github.com/jdg511/quadpreandrecorder"
- note added: "Rev C3: no test headers (J6/J7 removed - they forced every analog node across the board beside every clock). Probe at component pads."
- note added: "Teensy 4.1 records four mono WAV files over native SDIO and decodes the 48 kHz binaural monitor; USB-C = MTP file transfer + firmware updates."
- note added: "USB/POWER NOTE: CUT the Teensy VIN-VUSB link (the board powers VIN from +5V). USB data reaches the Teensy through TP1/TP2 wired to its underside USB-Device D+/D- pads; never plug the Teensy micro-B and J9 at the same time."
- note removed: "192 kHz / 24-bit capture • real-time binaural monitor • two-layer Rev B (Hammond 1590XX)"
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