File: hardware/review_outputs/QuadPreRecorder-unrouted.kicad_pcb (KiCad board)
At the start: 2 copper layers, 138 x 114 mm, 190 parts, among them J1 9V DC IN, J2 AMBISONIC MIC RJ45, J3 MSP3520 TFT 3.5IN 14PIN HEADER, J4 1/4in BINAURAL LINE OUT, J5 1/8in BINAURAL HEADPHONE OUT, J6 ANALOG TEST HEADER 2x13, J7 DIGITAL TEST HEADER 2x13, SW1 PAD -10dB, SW2 RECORD START/STOP, SW3 MASTER GAIN, SW4 TFT MENU NAV, U1 TPS62160DGK, U10 TPA6132A2, U2 TPS7A2033PDBV, U3 TLE2426ID, U4 CD4053BPW, U5 CD4053BPW, U6 OPA1654, U7 PCM1864DBT, U8 Teensy 4.1, U9 PCM5102A

Commit message: Rev B through Rev C3: 1590XX enclosure, CAT6 mic input, mic-mode rebuild, fab package, 3D enclosure models
- Rev B 2-layer, then Rev C/C2/C3 on Hammond 1590XX: USB-C power/data, capacitive MSP3526, TPA6130A2 headphone amp, LiPo + BQ24074, SW4 5-way encoder
- Mic-mode rebuild: per-channel bias off/5V/9V, cold-leg grounding, balanced inputs, SPICE CMRR fixes
- Enclosure fit recheck applied (J4/J5/J9 moves, SW2 replacement, front-wall LEDs); ADC test points; ADP7142 LDO swap
- PCBWay Rev C3 handoff package with 4-layer gerbers, BOM/CPL, best-source pricing
- Interactive labeled 3D enclosure models (1590XX as-built with logo + 1590F concept), labeled-views PDF, blog embed notes

Co-Authored-By: Claude Fable 5 <noreply@anthropic.com>
Claude-Session: https://claude.ai/code/session_01CTGyPyq5ASmP2zYeDmwtXd
Parts:
- removed C38: 1uF, Capacitor_SMD:C_0805_2012Metric
- removed C63: 100nF, Capacitor_SMD:C_0603_1608Metric
- removed J6: ANALOG TEST HEADER 2x13, Connector_PinHeader_2.54mm:PinHeader_2x13_P2.54mm_Vertical
- removed J7: DIGITAL TEST HEADER 2x13, Connector_PinHeader_2.54mm:PinHeader_2x13_P2.54mm_Vertical
- removed R68: 1k, Resistor_SMD:R_0603_1608Metric
- removed RV1: 10kA HEADPHONE VOLUME, QuadPreRecorder:RK097_Dual_Horizontal_NoEdgeGuide
- removed SW1: PAD -10dB, QuadPreRecorder:SW_Toggle_ESwitch_100SP_M7
- added C100: 100pF C0G, Capacitor_SMD:C_0603_1608Metric, B.Cu at (36.0, 104.4)
- added C101: 4.7uF 35V FILM, Capacitor_SMD:C_1812_4532Metric, B.Cu at (44.0, 85.5)
- added C102: 4.7uF 35V FILM, Capacitor_SMD:C_1812_4532Metric, B.Cu at (44.0, 91.8)
- added C103: 4.7uF 35V FILM, Capacitor_SMD:C_1812_4532Metric, B.Cu at (44.0, 98.1)
- added C104: 4.7uF 35V FILM, Capacitor_SMD:C_1812_4532Metric, B.Cu at (44.0, 104.4)
- added C105: 22pF C0G, Capacitor_SMD:C_0603_1608Metric, B.Cu at (63.0, 85.5)
- added C106: 22pF C0G, Capacitor_SMD:C_0603_1608Metric, B.Cu at (63.0, 91.8)
- added C107: 22pF C0G, Capacitor_SMD:C_0603_1608Metric, B.Cu at (63.0, 98.1)
- added C108: 22pF C0G, Capacitor_SMD:C_0603_1608Metric, B.Cu at (63.0, 104.4)
- added C109: 100nF, Capacitor_SMD:C_0603_1608Metric, F.Cu at (57.5, 58.5)
- added C110: 100nF, Capacitor_SMD:C_0603_1608Metric, F.Cu at (33.5, 60.5)
- added C74: 10uF 16V, Capacitor_SMD:C_1206_3216Metric, F.Cu at (18.5, 45.0)
- added C75: 100nF, Capacitor_SMD:C_0603_1608Metric, F.Cu at (17.0, 53.5)
- added C76: 10uF 25V, Capacitor_SMD:C_1206_3216Metric, F.Cu at (13.5, 37.5)
- added C77: 10uF 25V, Capacitor_SMD:C_1206_3216Metric, F.Cu at (18.5, 37.5)
- added C78: 100nF, Capacitor_SMD:C_0603_1608Metric, F.Cu at (48.0, 14.0)
- added C79: 47nF, Capacitor_SMD:C_0603_1608Metric, B.Cu at (15.0, 29.0)
- added C80: 4.7nF C0G, Capacitor_SMD:C_0603_1608Metric, F.Cu at (5.00, 45.0)
- added C81: 47pF C0G, Capacitor_SMD:C_0603_1608Metric, F.Cu at (9.00, 45.0)
- added C83: 2.2uF, Capacitor_SMD:C_0805_2012Metric, F.Cu at (5.50, 50.5)
- added C85: 10uF 25V, Capacitor_SMD:C_1206_3216Metric, F.Cu at (20.5, 18.5)
- added C86: 2.2uF 25V FILM, Capacitor_SMD:C_1210_3225Metric, F.Cu at (100.4, 55.7)
- added C87: 2.2uF 25V FILM, Capacitor_SMD:C_1210_3225Metric, F.Cu at (100.4, 59.1)
- added C88: 10uF 16V, Capacitor_SMD:C_1206_3216Metric, F.Cu at (17.0, 50.0)
- added C89: 100nF, Capacitor_SMD:C_0603_1608Metric, F.Cu at (132.0, 31.5)
- added C90: 10uF 10V, Capacitor_SMD:C_0805_2012Metric, F.Cu at (124.0, 15.0)
- added C91: 10uF 10V, Capacitor_SMD:C_0805_2012Metric, F.Cu at (135.0, 15.0)
- added C92: 10uF 10V, Capacitor_SMD:C_0805_2012Metric, F.Cu at (136.0, 24.5)
- added C93: 10nF, Capacitor_SMD:C_0603_1608Metric, B.Cu at (110.0, 36.0)
- added C94: 10nF, Capacitor_SMD:C_0603_1608Metric, B.Cu at (114.0, 36.0)
- added C95: 1uF 10V, Capacitor_SMD:C_0805_2012Metric, B.Cu at (92.5, 63.0)
- added C96: 4.7uF 10V, Capacitor_SMD:C_0805_2012Metric, B.Cu at (88.0, 63.0)
- added C97: 100pF C0G, Capacitor_SMD:C_0603_1608Metric, B.Cu at (36.0, 85.5)
- added C98: 100pF C0G, Capacitor_SMD:C_0603_1608Metric, B.Cu at (36.0, 91.8)
- added C99: 100pF C0G, Capacitor_SMD:C_0603_1608Metric, B.Cu at (36.0, 98.1)
- added D10: B340A 40V 3A, Diode_SMD:D_SMA, F.Cu at (52.0, 10.5)
- added D11: USBLC6-2SC6, Package_TO_SOT_SMD:SOT-23-6, F.Cu at (40.0, 12.8)
- added D12: B340A 40V 3A, Diode_SMD:D_SMA, F.Cu at (7.00, 37.5)
- added D13: 1N4148W, Diode_SMD:D_SOD-123, F.Cu at (104.0, 100.5)
- added D14: B340A 40V 3A, Diode_SMD:D_SMA, F.Cu at (131.0, 24.5)
- added D15: 1N4148W, Diode_SMD:D_SOD-123, F.Cu at (123.5, 28.2)
- added D16: 1N4148W, Diode_SMD:D_SOD-123, F.Cu at (128.3, 28.2)
- added D17: 1N4148W, Diode_SMD:D_SOD-123, F.Cu at (133.1, 28.2)
- added D18: 1N4148W, Diode_SMD:D_SOD-123, B.Cu at (98.0, 16.0)
- added D19: 1N4148W, Diode_SMD:D_SOD-123, B.Cu at (98.0, 20.0)
- added D20: PESD12VL1BA, Diode_SMD:D_SOD-323, B.Cu at (40.0, 85.5)
- added D21: PESD12VL1BA, Diode_SMD:D_SOD-323, B.Cu at (40.0, 91.8)
- added D22: PESD12VL1BA, Diode_SMD:D_SOD-323, B.Cu at (40.0, 98.1)
- added D23: PESD12VL1BA, Diode_SMD:D_SOD-323, B.Cu at (40.0, 104.4)
- added D24: BAT54, Diode_SMD:D_SOD-123, F.Cu at (34.0, 82.5)
- added F2: 2A PTC, Fuse:Fuse_1206_3216Metric, F.Cu at (52.0, 6.00)
- added J10: BATTERY 1S LiPo, Connector_JST:JST_PH_B2B-PH-K_1x02_P2.00mm_Vertical, B.Cu at (121.0, 109.5)
- added J9: USB-C POWER + DATA, Connector_USB:USB_C_Receptacle_HRO_TYPE-C-31-M-12, F.Cu at (40.0, 2.60)
- added K1: G6K-2F-Y 5VDC, Relay_SMD:Relay_DPDT_Omron_G6K-2F-Y, F.Cu at (113.0, 103.5)
- added L2: 10uH 2A, Inductor_SMD:L_Bourns_SRN6045TA, F.Cu at (18.0, 31.5)
- added Q1: 2N7002, Package_TO_SOT_SMD:SOT-23, F.Cu at (6.00, 58.0)
- added Q2: 2N7002, Package_TO_SOT_SMD:SOT-23, F.Cu at (104.0, 104.0)
- added Q3: AO3401A, Package_TO_SOT_SMD:SOT-23, F.Cu at (30.0, 67.0)
- added Q4: AO3401A, Package_TO_SOT_SMD:SOT-23, F.Cu at (30.0, 71.0)
- added Q5: 2N7002, Package_TO_SOT_SMD:SOT-23, F.Cu at (34.0, 64.5)
- added Q6: AO3401A, Package_TO_SOT_SMD:SOT-23, F.Cu at (34.0, 75.5)
- added Q7: 2N7002, Package_TO_SOT_SMD:SOT-23, F.Cu at (34.0, 79.5)
- added Q8: AO3401A, Package_TO_SOT_SMD:SOT-23, F.Cu at (38.0, 75.5)
- added Q9: 2N7002, Package_TO_SOT_SMD:SOT-23, F.Cu at (38.0, 79.5)
- added R100: 100k, Resistor_SMD:R_0603_1608Metric, F.Cu at (26.5, 70.9)
- added R101: 100k, Resistor_SMD:R_0603_1608Metric, F.Cu at (41.0, 77.1)
- added R102: 100R, Resistor_SMD:R_0603_1608Metric, F.Cu at (38.0, 82.5)
- added R103: 100k, Resistor_SMD:R_0603_1608Metric, F.Cu at (26.5, 74.0)
- added R104: 100k BLEED, Resistor_SMD:R_0603_1608Metric, F.Cu at (26.5, 77.1)
- added R106: 10k, Resistor_SMD:R_0603_1608Metric, F.Cu at (34.5, 68.5)
- added R107: 100R, Resistor_SMD:R_0603_1608Metric, F.Cu at (38.0, 68.5)
- added R108: 100k, Resistor_SMD:R_0603_1608Metric, F.Cu at (34.5, 71.5)
- added R110: 100R RF, Resistor_SMD:R_0603_1608Metric, B.Cu at (32.0, 85.5)
- added R111: 100R RF, Resistor_SMD:R_0603_1608Metric, B.Cu at (32.0, 91.8)
- added R112: 100R RF, Resistor_SMD:R_0603_1608Metric, B.Cu at (32.0, 98.1)
- added R113: 100R RF, Resistor_SMD:R_0603_1608Metric, B.Cu at (32.0, 104.4)
- added R114: 1M, Resistor_SMD:R_0603_1608Metric, B.Cu at (48.0, 85.5)
- added R115: 1M, Resistor_SMD:R_0603_1608Metric, B.Cu at (48.0, 91.8)
- added R116: 1M, Resistor_SMD:R_0603_1608Metric, B.Cu at (48.0, 98.1)
- added R117: 1M, Resistor_SMD:R_0603_1608Metric, B.Cu at (48.0, 104.4)
- added R118: 10k 0.1%, Resistor_SMD:R_0603_1608Metric, B.Cu at (52.0, 85.5)
- added R119: 10k 0.1%, Resistor_SMD:R_0603_1608Metric, B.Cu at (52.0, 91.8)
- added R120: 10k 0.1%, Resistor_SMD:R_0603_1608Metric, B.Cu at (52.0, 98.1)
- added R121: 10k 0.1%, Resistor_SMD:R_0603_1608Metric, B.Cu at (52.0, 104.4)
- added R122: 90.9k 0.1%, Resistor_SMD:R_0603_1608Metric, B.Cu at (56.0, 85.5)
- added R123: 90.9k 0.1%, Resistor_SMD:R_0603_1608Metric, B.Cu at (56.0, 91.8)
- added R124: 90.9k 0.1%, Resistor_SMD:R_0603_1608Metric, B.Cu at (56.0, 98.1)
- added R125: 90.9k 0.1%, Resistor_SMD:R_0603_1608Metric, B.Cu at (56.0, 104.4)
- added R126: 100k, Resistor_SMD:R_0603_1608Metric, B.Cu at (50.0, 85.5)
- added R127: 100k, Resistor_SMD:R_0603_1608Metric, B.Cu at (50.0, 91.8)
- added R128: 100k, Resistor_SMD:R_0603_1608Metric, B.Cu at (50.0, 98.1)
- added R129: 100k, Resistor_SMD:R_0603_1608Metric, B.Cu at (50.0, 104.4)
- added R130: 130k, Resistor_SMD:R_0603_1608Metric, F.Cu at (13.3, 48.6)
- added R131: 20k, Resistor_SMD:R_0603_1608Metric, F.Cu at (13.3, 52.4)
- added R75: 5.1k, Resistor_SMD:R_0603_1608Metric, F.Cu at (33.0, 9.00)
- added R76: 5.1k, Resistor_SMD:R_0603_1608Metric, F.Cu at (47.0, 9.00)
- added R77: 100k, Resistor_SMD:R_0603_1608Metric, F.Cu at (56.0, 14.0)
- added R78: 47k, Resistor_SMD:R_0603_1608Metric, F.Cu at (52.0, 14.0)
- added R79: 10k, Resistor_SMD:R_0603_1608Metric, F.Cu at (17.0, 41.5)
- added R80: 75k, Resistor_SMD:R_0603_1608Metric, F.Cu at (5.00, 41.5)
- added R81: 10k, Resistor_SMD:R_0603_1608Metric, F.Cu at (9.00, 41.5)
- added R82: 80.6k, Resistor_SMD:R_0603_1608Metric, F.Cu at (13.0, 41.5)
- added R83: 10k, Resistor_SMD:R_0603_1608Metric, F.Cu at (18.5, 57.5)
- added R84: 100R, Resistor_SMD:R_0603_1608Metric, F.Cu at (100.0, 104.0)
- added R85: 100k, Resistor_SMD:R_0603_1608Metric, F.Cu at (100.0, 107.5)
- added R86: 1M, Resistor_SMD:R_0603_1608Metric, F.Cu at (30.0, 74.5)
- added R87: 1M, Resistor_SMD:R_0603_1608Metric, F.Cu at (30.0, 77.5)
- added R88: 1M, Resistor_SMD:R_0603_1608Metric, F.Cu at (136.5, 28.5)
- added R89: 1M, Resistor_SMD:R_0603_1608Metric, F.Cu at (124.0, 31.5)
- added R90: 1M, Resistor_SMD:R_0603_1608Metric, F.Cu at (128.0, 31.5)
- added R91: 1.1k ILIM, Resistor_SMD:R_0603_1608Metric, F.Cu at (123.5, 20.5)
- added R92: 1.2k ISET, Resistor_SMD:R_0603_1608Metric, F.Cu at (127.0, 20.5)
- added R93: 10k TS, Resistor_SMD:R_0603_1608Metric, F.Cu at (130.5, 20.5)
- added R94: 100k, Resistor_SMD:R_0603_1608Metric, F.Cu at (134.0, 20.5)
- added R95: 100k, Resistor_SMD:R_0603_1608Metric, F.Cu at (124.0, 24.5)
- added R96: 10k, Resistor_SMD:R_0603_1608Metric, B.Cu at (102.0, 36.0)
- added R97: 10k, Resistor_SMD:R_0603_1608Metric, B.Cu at (106.0, 36.0)
- added R98: 100k, Resistor_SMD:R_0603_1608Metric, F.Cu at (41.0, 74.0)
- added R99: 100R, Resistor_SMD:R_0603_1608Metric, F.Cu at (41.0, 80.2)
- added TP1: USB D+ WIRE TO TEENSY, TestPoint:TestPoint_Pad_2.0x2.0mm, B.Cu at (56.5, 18.0)
- added TP10: DAC_LRCLK, TestPoint:TestPoint_Pad_1.5x1.5mm, B.Cu at (90.5, 42.2)
- added TP11: DAC_DIN, TestPoint:TestPoint_Pad_1.5x1.5mm, B.Cu at (94.5, 42.2)
- added TP12: +3V3_DC, TestPoint:TestPoint_Pad_1.5x1.5mm, B.Cu at (84.0, 63.0)
- added TP13: GND, TestPoint:TestPoint_Pad_1.5x1.5mm, B.Cu at (82.5, 42.2)
- added TP14: GND, TestPoint:TestPoint_Pad_1.5x1.5mm, B.Cu at (81.0, 59.5)
- added TP2: USB D- WIRE TO TEENSY, TestPoint:TestPoint_Pad_2.0x2.0mm, B.Cu at (56.5, 21.5)
- added TP3: ADC_MCLK, TestPoint:TestPoint_Pad_1.5x1.5mm, B.Cu at (84.5, 36.5)
- added TP4: ADC_BCLK, TestPoint:TestPoint_Pad_1.5x1.5mm, B.Cu at (88.0, 36.5)
- added TP5: ADC_LRCLK, TestPoint:TestPoint_Pad_1.5x1.5mm, B.Cu at (91.5, 36.5)
- added TP6: ADC_TDM, TestPoint:TestPoint_Pad_1.5x1.5mm, B.Cu at (95.0, 36.5)
- added TP7: ADC_DOUT2, TestPoint:TestPoint_Pad_1.5x1.5mm, B.Cu at (98.5, 36.5)
- added TP8: GND, TestPoint:TestPoint_Pad_1.5x1.5mm, B.Cu at (81.0, 36.5)
- added TP9: DAC_BCLK, TestPoint:TestPoint_Pad_1.5x1.5mm, B.Cu at (86.5, 42.2)
- added U11: TPS61175PWP, Package_SO:Texas_HTSSOP-14-1EP_4.4x5mm_P0.65mm_EP3.4x5mm_Mask3.155x3.255mm, F.Cu at (9.50, 31.5)
- added U12: ADP7142AUJZ, Package_TO_SOT_SMD:TSOT-23-5, F.Cu at (9.50, 50.5)
- added U13: BQ24074RGT, Package_DFN_QFN:VQFN-16-1EP_3x3mm_P0.5mm_EP1.68x1.68mm, F.Cu at (129.5, 16.5)
- added U14: TPS7A2033PDBV, Package_TO_SOT_SMD:SOT-23-5, B.Cu at (88.0, 59.5)
- added U15: CD4053BPW, Package_SO:TSSOP-16_4.4x5mm_P0.65mm, F.Cu at (40.5, 63.0)
- added U16: OPA1654, Package_SO:TSSOP-14_4.4x5mm_P0.65mm, F.Cu at (52.0, 61.5)
- C17, C18, C19, C20, C25, C26, C27, C28: value 4.7uF 16V -> 4.7uF 35V FILM; footprint Capacitor_SMD:C_1206_3216Metric -> Capacitor_SMD:C_1812_4532Metric
- C53: footprint Capacitor_SMD:C_0805_2012Metric -> Capacitor_SMD:C_0603_1608Metric; moved to B.Cu
- C54, C55, C56, C64: moved to B.Cu
- C57: value 680nF X7R -> 2.2uF 25V FILM; footprint Capacitor_SMD:C_0805_2012Metric -> Capacitor_SMD:C_1210_3225Metric
- C58: value 680nF X7R -> 2.2uF 25V FILM; footprint Capacitor_SMD:C_0603_1608Metric -> Capacitor_SMD:C_1210_3225Metric
- C60, C61, C65: value 2.2uF -> 1uF
- D1: value SS14 -> B340A 40V 3A
- D4, D5: footprint LED_SMD:LED_0603_1608Metric -> LED_THT:LED_D3.0mm_Horizontal_O1.27mm_Z6.0mm
- H5, H6, H7, H8: value M3 TFT MSP3520 PROVISIONAL-VERIFY -> M3 TFT MSP3526 92x49.5 VERIFY
- J3: value MSP3520 TFT 3.5IN 14PIN HEADER -> MSP3526 TFT 3.5IN 14PIN SOCKET; footprint Connector_PinHeader_2.54mm:PinHeader_1x14_P2.54mm_Vertical -> Connector_PinSocket_2.54mm:PinSocket_1x14_P2.54mm_Vertical
- R42: value 100k -> 100R
- R43: value 47k -> 100k
- SW2: footprint Button_Switch_THT:SW_PUSH-12mm -> Button_Switch_THT:SW_PUSH_6mm
- SW4: footprint QuadPreRecorder:SW_Nav_ALPS_SKQUCAA010 -> QuadPreRecorder:SW_Nav5_ALPS_RKJXT1F42001
- U10: value TPA6132A2 -> TPA6130A2RTJ; footprint Package_DFN_QFN:WQFN-16-1EP_3x3mm_P0.5mm_EP1.6x1.6mm -> Package_DFN_QFN:WQFN-20-1EP_4x4mm_P0.5mm_EP2.7x2.7mm
- moved J1 133.1 mm to (17.5, 8.20), turned to 180 degrees
- moved C1 131.2 mm to (17.0, 24.5)
- moved F1 125.5 mm to (7.00, 18.5), turned to 0 degrees
- moved D1 115.3 mm to (14.5, 18.5), turned to 0 degrees
- moved D2 111.8 mm to (8.00, 23.5), turned to 0 degrees
- moved J3 98.6 mm to (25.0, 19.2), turned to 0 degrees
- moved C40 27.5 mm to (82.8, 47.7)
- moved C39 27.3 mm to (83.0, 45.9)
- moved C57 27.1 mm to (106.4, 54.6)
- moved C58 25.5 mm to (106.4, 60.2)
- moved FID4 22.8 mm to (30.0, 22.0)
- moved FID1 22.4 mm to (30.0, 18.0)
- moved C61 16.6 mm to (110.3, 51.8), turned to 90 degrees
- moved U7 15.5 mm to (83.5, 49.5)
- moved C55 15.4 mm to (99.9, 55.0)
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Connections:
- C1 pad 1: +9V -> VBOOST_IN
- C2 pad 1: +9V -> +10V5
- C3 pad 1: +9V -> +10V5
- C33 pad 1: PAD_SENSE -> PAD_SELECT
- C44 pad 1: +3V3_D -> +3V3_DC
- C45 pad 1: +3V3_D -> +3V3_DC
- C56 pad 1: +3V3_D -> +3V3_DC
- C57 pad 1: HP_VOL_L -> LINE_L
- C58 pad 1: HP_VOL_R -> LINE_R
- C61 pad 1: HPVDD -> +5V
- D1 pad 1: +9V -> VBOOST_IN
- D2 pad 1: +9V -> VBOOST_IN
- J2 pad 2: GND -> FLU_RAWC
- J2 pad 5: GND -> BLD_RAWC
- J2 pad 6: GND -> FRD_RAWC
- J2 pad 8: GND -> BRU_RAWC
- J3 pad 10: SPI_SCK -> I2C_SCL
- J3 pad 11: TOUCH_CS -> CTP_RST
- J3 pad 12: SPI_MOSI -> I2C_SDA
- J3 pad 13: SPI_MISO -> TOUCH_IRQ
- J3 pad 14: TOUCH_IRQ -> (no net)
- J4 pad R: LINE_R -> LINE_JACK_R
- J4 pad T: LINE_L -> LINE_JACK_L
- R26 pad 2: VREF -> FLU_CPRE
- R27 pad 2: VREF -> FRD_CPRE
- R28 pad 2: VREF -> BLD_CPRE
- R29 pad 2: VREF -> BRU_CPRE
- R42 pad 1: PAD_SELECT -> PAD_CTRL
- R42 pad 2: PAD_SENSE -> PAD_CTRL_G
- R43 pad 1: PAD_SENSE -> PAD_CTRL_G
- R67 pad 1: +9V -> BIAS_SRC
- SW2 pad 1: REC_BUTTON -> REC_SW
- SW3 pad S1: GAIN_PUSH -> GAIN_SW
- SW4 pad 5: NAV_RIGHT -> NAV_PUSH
- SW4 pad 6: NAV_PUSH -> GND
- U1 pad 2: +9V -> +10V5
- U1 pad 3: +9V -> +10V5
- U10 pad 11: HP_CPP -> HP_OUT_R
- U10 pad 12: HPVDD -> +5V
- U10 pad 13: HP_ENABLE -> GND
- U10 pad 14: +5V -> HP_OUT_L
- U10 pad 15: GND -> HP_VSS
- U10 pad 16: HP_OUT_L -> HP_VSS
- U10 pad 17: GND -> HP_CPN
- U10 pad 2: GND -> HP_INP_L
- U10 pad 4: HP_IN_R -> HP_INP_R
- U10 pad 5: HP_OUT_R -> HP_IN_R
- U10 pad 6: +3V3_D -> HP_ENABLE
- U10 pad 7: GND -> I2C_SDA
- U10 pad 8: HP_VSS -> I2C_SCL
- U10 pad 9: HP_CPN -> GND
- U4 pad 3: (no net) -> GND
- U4 pad 4: (no net) -> FLU_MICC
- U4 pad 9: GND -> COLD_SEL
- U5 pad 3: (no net) -> GND
- U5 pad 4: (no net) -> BLD_MICC
- U5 pad 9: GND -> COLD_SEL
- U7 pad 13: +3V3_D -> +3V3_DC
- U7 pad 14: +3V3_D -> +3V3_DC
- U7 pad 5: ADC_MICBIAS -> (no net)
- U8 pad 0: (no net) -> MIC5_CTRL
- U8 pad 1: (no net) -> MIC9_CTRL
- U8 pad 14: (no net) -> CTP_RST
- U8 pad 15: (no net) -> VBUS_SENSE
- U8 pad 16: (no net) -> BAT_SENSE
- U8 pad 17: (no net) -> CHG_STAT_N
- U8 pad 24: TOUCH_CS -> KEEP_ON
- U8 pad 25: (no net) -> PGOOD_N
- U8 pad 26: (no net) -> NAV_ENC_A
- U8 pad 27: (no net) -> NAV_ENC_B
- U8 pad 32: PAD_SENSE -> PAD_CTRL
- U8 pad 3V3B: +3V3_D -> (no net)
- U8 pad 41: (no net) -> COLD_CTRL
- U8 pad 5: (no net) -> LINE_MUTE
- U9 pad 20: +3V3_D -> +3V3_DC
Routing:
- added copper zone on In1.Cu, net GND
- added copper zone on In2.Cu, net GND
Other:
- outline, holes or cut-outs redrawn
- copper layers 2 -> 4
- board text added: "3.5in MSP3526 MODULE ENVELOPE 98x55.5 - VERIFY MODULE"
- board text added: "BATT J10 + LiPo 906090 UNDER RIGHT HALF"
- board text added: "CHG"
- board text added: "K1 LINE MUTE"
- board text added: "MSP3526 PIN1"
- board text added: "PWR: HOLD REC+GAIN 2s"
- board text added: "TEENSY 4.1 ON BOTTOM - CUT VIN/VUSB LINK"
- board text added: "TP1 D+ / TP2 D- -> TEENSY USB PADS"
- board text added: "USB-C 5V"
- board text added: "jdg511 QUAD PRE RECORDER REV C HAMMOND 1590XX"
- board text removed: "3.5in MSP3520 MODULE ENVELOPE - VERIFY MODULE"
- board text removed: "MSP3520 TFT 1..14"
- board text removed: "PAD"
- board text removed: "TEENSY 4.1 ON BOTTOM - CUT VIN/VUSB FOR DUAL POWER"
- board text removed: "VOL"
- board text removed: "jdg511 QUAD PRE RECORDER REV B HAMMOND 1590XX"
